Commit message: added g1 primitive collisions model with multi-height knee knocker curriculum

File: source/my_usds/navy_door.urdf (robot description, URDF)
Before this commit: robot navy_door, 1 links, 0 joints
Links:
- link door_frame: geometry collision box size=1.118 0.05 2.2; collision box size=1.118 0.05 2.2
